File: hardware/cpu_luefter_ansteuerung.sch (KiCad schematic (older format))
At the start: 24 parts, among them J1 Power 12V DC, J2 ISP, J3 CPU Lüfter, Q1 BC337, SW1 SW_Push, U1 L7805, U2 ATtiny24A-PU, U3 74HC595, U4 KCSA02-123

Commit message: J3 Footprint geändert
Parts:
- J3: footprint Connector_PinHeader_1.27mm:PinHeader_1x04_P1.27mm_Vertical -> Connector_PinSocket_2.54mm:PinSocket_1x04_P2.54mm_Vertical
Changed lines of the file:
@@
 EESchema Schematic File Version 4
 LIBS:cpu_luefter_ansteuerung-cache
-EELAYER 29 0
+EELAYER 30 0
 EELAYER END
 $Descr A4 11693 8268
@@
 F 0 "J3" H 9980 4892 50  0000 L CNN
 F 1 "CPU Lüfter" H 9980 4801 50  0000 L CNN
-F 2 "Connector_PinHeader_1.27mm:PinHeader_1x04_P1.27mm_Vertical" H 9900 4900 50  0001 C CNN
+F 2 "Connector_PinSocket_2.54mm:PinSocket_1x04_P2.54mm_Vertical" H 9900 4900 50  0001 C CNN
 F 3 "~" H 9900 4900 50  0001 C CNN
 	1    9900 4900
